File: src/schematics/kitchen-led-strips/kitchen-led-strips.kicad_sch (KiCad schematic)
At the start: 31 parts, among them U1 AP62150WU, U2 PIC16F15355-I/MV

Commit message: Further elaboration of the schematic.
Parts:
- added C? (x7): 2.2μF, restall-generic-capacitors:unpolarised-nominal-0603-1608, symbol restall-generic-capacitors:capacitor-unpolarised
- added C?: 10μF, restall-generic-capacitors:unpolarised-nominal-1206-3216, symbol restall-generic-capacitors:capacitor-unpolarised
- added CONN1: PSG01593, restall-generic-connectors:th-header-1x2-2.54mm-vertical, symbol restall-generic-connectors:circular-4p-shield-male
- added CONN1a, CONN2a: DNP, restall-generic-connectors:th-header-1x2-2.54mm-vertical, symbol restall-generic-connectors:header-1x2
- added CONN2: PSG01593, symbol restall-generic-connectors:circular-4p-shield-female
- added CONN2b: DNP, restall-generic-connectors:th-header-1x4-2.54mm-vertical, symbol restall-generic-connectors:header-1x4
- added CONN?: S5B-PH-K-S, restall-manufacturer-jst:S5B-PH-K-?, symbol restall-generic-connectors:header-1x5
- added CONN?: header-2x13-row, restall-generic-connectors:th-header-2x13-2.54mm-row-horizontal-shrouded, symbol restall-generic-connectors:header-2x13-row
- added D? (x8): BZA856AVL,115, restall-generic-sot:SOT-353, symbol restall-manufacturer-nexperia:BZA856AVL,115
- added Q? (x4): BC847BS, restall-manufacturer-diodes-inc:SOT-363, symbol restall-manufacturer-diodes-inc:BC847BS
- added R? (x6): 634Ω, restall-generic-resistors:nominal-0402-1005, symbol restall-generic-resistors:resistor
- added R? (x2): 91Ω, restall-generic-resistors:nominal-0402-1005, symbol restall-generic-resistors:resistor
- added R? (x5): 4.7kΩ, restall-generic-resistors:nominal-0402-1005, symbol restall-generic-resistors:resistor
- added R?: 7.5Ω, restall-generic-resistors:nominal-0603-1608, symbol restall-generic-resistors:resistor
- added R?: 470Ω, restall-generic-resistors:nominal-0402-1005, symbol restall-generic-resistors:resistor
- R?: value 470Ω -> 634Ω; Label 470Ω±1% 0.0625W -> 634Ω±1% 0.0625W; Manufacturer (none) -> Yageo; ManufacturerPartNumber (none) -> RC0402FR-07634RL
Connections:
- net +12V_{dc}: now also CONN1.1 (P1), CONN1a.1 (P1)
- net +5Vdc: now also C?.1, C?.1, C?.1, C?.1, C?.1, C?.1, CONN?.11 (P11), CONN?.17 (P17), CONN?.2 (P2), CONN?.4 (P4), CONN?.5 (P5), R?.1, R?.1, R?.1
- net GND: now also C?.2, C?.2, C?.2, C?.2, C?.2, C?.2, C?.2, C?.2, CONN1.2 (P2), CONN1.3 (P3), CONN1.4 (P4), CONN1a.2 (P2), CONN2.2 (P2), CONN2b.3 (P3), CONN?.10 (P10), CONN?.12 (P12), CONN?.14 (P14), CONN?.16 (P16), CONN?.18 (P18), CONN?.20 (P20), CONN?.22 (P22), CONN?.24 (P24), CONN?.26 (P26), CONN?.3 (P3), CONN?.4 (P4), CONN?.6 (P6), CONN?.8 (P8), D?.2 (A), D?.2 (A), D?.2 (A), D?.2 (A), D?.2 (A), D?.2 (A), D?.2 (A), Q?.1 (E), Q?.4 (E), Q?.4 (E), R?.2
- net MCU_ICSP_{CLK}: now also CONN?.1 (P1), D?.1 (K), R?.2; no longer U2.24 (RB6)
- net MCU_ICSP_{DAT}: now also CONN?.2 (P2), D?.3 (K), R?.2; no longer U2.25 (RB7)
- net VLED_{EN}: now also U2.23 (RB5); no longer U2.15 (RC7)
- net VLED_{PG}: now also U2.22 (RB4); no longer U2.14 (RC6)
- net ~{MCU_MCLR}: now also CONN?.5 (P5), D?.4 (K)
- net at R?.1: now also U2.4 (RA5); no longer U2.13 (RC5)
- net LED_{D1}: now reaches R?.2, R?.2, R?.2
- net LED_{D1}: now also CONN2.4 (P4), CONN2b.4 (P4)
- net at R?.1: now also U2.2 (RA3); no longer U2.11 (RC3)
- net at U2.9 (RC1): now also R?.2; no longer R?.1
- net LED_{D0}: now reaches R?.2, R?.2, R?.2
- net LED_{D0}: now also CONN2.3 (P3), CONN2b.1 (P1)
- net VLED: now reaches C?.1, R?.2, U?.7 (V_{OUT}), U?.8 (V_{OUT})
- net VLED: now also CONN2.1 (P1), CONN2a.1 (P1)
- net at R?.1: now also U2.27 (RA0); no longer U2.8 (RC0)
- net at U2.12 (RC4): now also R?.1; no longer R?.1
- net at U2.10 (RC2): now also R?.2; no longer R?.1
- net at U2.1 (RA2): now also R?.1
- net at U2.19 (RB1): now also R?.2
- net at U2.20 (RB2): now also R?.2
- net at U2.28 (RA1): now also R?.1
- net at U2.3 (RA4): now also R?.1
- net at U2.6 (RA7): now also R?.2
- net IR_REC: now reaches U2.7 (RA6)
- net IR_REC: now also CONN?.1 (P1), D?.3 (K), R?.2
- new net: R?.2, U2.11 (RC3)
- new net: R?.1, U2.13 (RC5)
- new net: Q?.5 (B), R?.2
- new net: R?.1, U2.24 (RB6)
- new net: R?.1, U2.25 (RB7)
- new net: Q?.2 (B), R?.2
- new net: C?.1, CONN2a.2 (P2)
- new net: Q?.2 (B), Q?.3 (C), R?.1
- new net: Q?.1 (E), Q?.5 (B), R?.1
- new net: C?.1, CONN2b.2 (P2)
- new net: R?.2, U2.8 (RC0)
- new net GPIO_{0}: CONN?.25 (P25), R?.1
- new net GPIO_{1}: CONN?.23 (P23), R?.1
- new net GPIO_{2}: CONN?.21 (P21), R?.1
- new net GPIO_{3}: CONN?.19 (P19), R?.1
- new net GPOC_{0}: CONN?.15 (P15), Q?.6 (C)
- new net GPOC_{1}: CONN?.13 (P13), Q?.3 (C)
- new net IR_LED: CONN?.3 (P3), D?.1 (K), Q?.6 (C)
- new net I^{2}C_SCL: CONN?.9 (P9), D?.4 (K), R?.1, R?.2
- new net I^{2}C_SDA: CONN?.7 (P7), D?.5 (K), R?.1, R?.2
Other:
- note added: "Connect pin 2 direct to pin 2 on CONN1 to prevent high DC return currents flowing on PCB signal ground."
- note added: "Current source for roughly 87mA; 75mA-96mA over temperature"
- note added: "Ensure 2.5mm^{2} hole sizes for CONN1a and CONN2a."
- note added: "If cable length requires it then place a further 4.7kΩ (externally) in parallel with R? and R? to increase the I^{2}C drive strength to about its maximum"
- note added: "Keep high current traces to minimal lengths on PCB - route off-board with discrete wires, direct to connectors."
- note added: "Maximum LED strip is 5m@14.4W/m Input is 12V_{dc}±10%, maximum 7A."
- note added: "Pin 2 of CONN2a provides flexibility in routing ground return currents."
- note added: "Pins 2 and 3 provide flexibility in routing ground return currents for the fast LED_{Dx} edges whilst avoiding potentially large DC return."
- note added: "Pins 3 and 4 allow chassis-to-signal-ground connection at a single point inside the connector, if necessary."
- note added: "TODO: ADD 680R RESISTORS IN APPROPRIATE PLACES, TOO..."
- note added: "TODO: ALL 0402 R ASSUMED TO BE 0.0625W, 100ppm, +/-1%, THICK ALL 0603 R ASSUMED TO BE 0.1W, 100ppm, +/-1% THICK ALL 0805 R ASSUMED TO BE 0.25W, 100ppm, +/-1% THICK"
- note added: "TODO: TRANSIENT SUPPRESSION"
- note added: "TODO: TVS FOR GPIO LINES TVS FOR GPOC LINES"
- note added: "TODO: TVS FOR LED LINES"
- note added: "TODO: WHAT TO DO WITH THIS ?"
- note removed: "RC0-5 can be PWM out to LEDs USE TWO HOLES AND SOLDER WIRES DIRECTLY TO CHASSIS CONNECTOR; LEAVE LONG ENOUGH TO BE ABLE TO PULL OFF THE FACE PLATE."
- note removed: "TODO: CONNECTOR"
- note removed: "TODO: DO NOT CONNECT CHASSIS AND GND - THIS CAN BE DONE AT THE CONNECTOR CONNECT TWO PINS OF INPUT CONNECTOR TO +12V and 0V CONNECT TWO PINS OF INPUT CONNECTOR TO ENCLOSURE; THAT WAY THE CONNECTOR CAN MAKE THE GND-SHIELD CONNECTION IF NECESSARY"
- note removed: "TODO: GPIO CONNECTOR; ADD 10uF 25V FOR +5V OUT"
- note removed: "TODO: KEEP PCB TRACK FOR HIGH CURRENT VERY SHORT. WILL PREVENT GND DROP AND HEATING, PLUS THE CABLE FROM THE CONNECTOR NEEDS TO BE LONG ANYWAY TO FACILITATE THE FRONT PLATE BEING SEPARATED FROM THE ENCLOSURE JOIN THE CABLE TO A THROUGH-HOLE CLOSE TO THE LOAD SWITCH'S VIN PIN"
- note removed: "TODO: RA0-7 ARE GPIO ROUTE TO 2-ROW HEADER ALONG WITH +5V AND LOTS OF GND"
- note removed: "TODO: RB4 AND RB5 - WHAT TO DO WITH THOSE ? ROUTING WILL BE PROBLEMATIC WITHOUT JUMPERS. TEST POINTS ?"
- note removed: "TODO: THESE ARE I^{2}C OUTPUTS - SEPARATE 3-PIN HEADER ?"
- note removed: "TODO: TO /MCLR OUTPUT, ALONG WITH ICSPDAT, ICSPCLK, VDD AND VSS (PICKIT PINOUT)"
- moved on the sheet: C?, L?, R?, U1, U2, U?

Commit message: Finalised the schematic.  Ready for part numbering and checking.
Parts:
- added C? (x2): 2.2μF, restall-generic-capacitors:unpolarised-nominal-0603-1608, symbol restall-generic-capacitors:capacitor-unpolarised
- added CONN?: DNP, restall-generic-connectors:th-header-1x4-2.54mm-vertical, symbol restall-generic-connectors:header-1x4
- added CONN?: DNP, restall-generic-connectors:th-header-1x3-2.54mm-vertical, symbol restall-generic-connectors:header-1x3
- added D? (x12): BZA856AVL,115, restall-generic-sot:SOT-353, symbol restall-manufacturer-nexperia:BZA856AVL,115
- added R?: 634Ω, restall-generic-resistors:nominal-0402-1005, symbol restall-generic-resistors:resistor
- R? (x8): value 91Ω -> 100Ω; Label 91Ω±1% 0.0625W -> 100Ω±1% 0.0625W
- R?: value 4.7kΩ -> 10kΩ
Connections:
- net +5Vdc: now also D?.5 (K), C?.1, C?.1, CONN?.1 (P1), CONN?.1 (P1), D?.4 (K), D?.4 (K), D?.5 (K), D?.5 (K)
- net GND: now also D?.2 (A), C?.2, C?.2, CONN?.3 (P3), CONN?.3 (P3), D?.2 (A), D?.2 (A), D?.2 (A), D?.2 (A), D?.2 (A), D?.2 (A), D?.2 (A), D?.2 (A), D?.2 (A), D?.2 (A), D?.2 (A), D?.2 (A)
- net GPIO_{0}: now also D?.1 (K)
- net GPIO_{1}: now also D?.3 (K)
- net GPIO_{2}: now also D?.4 (K)
- net GPIO_{3}: now also D?.5 (K)
- net GPOC_{0}: now also D?.3 (K)
- net GPOC_{1}: now also D?.1 (K)
- net IR_REC: now also R?.2; no longer U2.7 (RA6)
- net LED_{D0}: now also D?.3 (K)
- net LED_{D1}: now also D?.1 (K)
- net DEBUG_{1}: now reaches U2.14 (RC6)
- net DEBUG_{1}: now also CONN?.2 (P2)
- net DEBUG_{2}: now reaches U2.15 (RC7)
- net DEBUG_{2}: now also CONN?.4 (P4)
- net DEBUG_{0}: now reaches U2.18 (RB0)
- net DEBUG_{0}: now also CONN?.2 (P2)
- new net: R?.1, U2.7 (RA6)
Other:
- note added: "Unless otherwise specified: All resistors are thick-film ±1% ±100ppm All 0402 resistors are 0.0625W, 0603 are 0.1W and 0805 are 0.25W All unpolarised capacitors are MLCC ±10% with X7R tempco"
- note added: "Z_{CABLE} ~40Ω Z_{PIC} termination simulated using IBIS."
- note removed: "At V_{DD}=5.5V: Z_{IOL} ~15Ω Z_{IOH} ~36Ω Z_{IO} ~27Ω Z_{CABLE} ~40Ω"
- note removed: "TODO: ADD 680R RESISTORS IN APPROPRIATE PLACES, TOO..."
- note removed: "TODO: ALL 0402 R ASSUMED TO BE 0.0625W, 100ppm, +/-1%, THICK ALL 0603 R ASSUMED TO BE 0.1W, 100ppm, +/-1% THICK ALL 0805 R ASSUMED TO BE 0.25W, 100ppm, +/-1% THICK"
- note removed: "TODO: PIC TO SHUTDOWN SWITCH IF VIN > 13.5V; IT CAN WITHSTAND 18V BUT IT'S NOT DESIGNED FOR > 13.5V..."
- note removed: "TODO: TRANSIENT SUPPRESSION"
- note removed: "TODO: TVS FOR GPIO LINES TVS FOR GPOC LINES"
- note removed: "TODO: TVS FOR LED LINES"
- note removed: "TODO: USE 5V DIVIDER ON RB0 TO ARRIVE AT THRESHOLD FOR 13.5V ON VIN SO THAT IT CAN BE USED AS A COMPARATOR TRIGGER"
- note removed: "TODO: WHAT TO DO WITH THIS ?"
- moved on the sheet: C?, CONN1, CONN?, D?A, D?B, D?C, D?D, Q?A, Q?B, R?, U2

Commit message: Schematic tweaks and checks.  Added some TODOs for tomorrow.
Parts:
- added FB1: HI0805R800R-10, restall-manufacturer-laird:FB0805, symbol restall-manufacturer-laird:HI0805R800R-10
- CONN1a, CONN2a, CONN2b: now left out of the parts list
- CONN5, CONN6: renamed from CONN?; now left out of the parts list
- L1: renamed from L?; Label 3.5A_{RMS} / 4.4A_{SAT}, 24mΩ±20% @ DC -> 3.3μH±20%, 3.5A_{RMS} / 4.4A_{SAT}, 24mΩ±20% @ DC
- R14, R15, R16, R17, R18, R19, R20, R21: renamed from R?; value 100Ω -> 91Ω; Label 100Ω±1% 0.0625W -> 91Ω±1% 0.0625W
- gave numbers to parts that had none: 55
- renumbered U1 to U2, U2 to U3
Connections:
- net +12V_{dc}: now also FB1.2 (P2); no longer C1.1, CONN1.1 (P1), CONN1a.1 (P1), R1.1, U1.1 (V_{IN}), U1.9 (V_{IN})
- net GND: no longer CONN1.2 (P2), CONN2.2 (P2)
- new net: C1.1, CONN1.1 (P1), CONN1a.1 (P1), FB1.1 (P1), R1.1, U1.1 (V_{IN}), U1.9 (V_{IN})
- new net: CONN1.2 (P2), CONN2.2 (P2)
Other:
- note added: "High-Voltage Programming not supported. Transient protection limits bandwidth so keep ICSP clock at 1MHz or less."
- note added: "If cable length requires it then place a further 4.7kΩ (externally) in parallel with R22 and R23 to increase the I^{2}C drive strength to about its maximum. A compromise between meeting I^{2}C V_{IL} and circuit simplicity has been made for ESD protection of these pins. Violation of the PIC's I_{K} clamping current (20mA) may occur."
- note added: "R14-19"
- note added: "R20-21"
- note added: "R27-30"
- note added: "R9-10"
- note added: "TODO: NEEDS PROTECTION DIODE FROM C13 -> VCC, SINCE +12V COULD BE POWERED WHILST SMPS IS OFF !"
- note added: "TODO: PART SELECTION STILL NEEDS TO BE DONE."
- note added: "TODO: PIC BLOCK AND BLOCK TO RIGHT STILL TO REVIEW SMPS AND INPUT BLOCKS HAVE BEEN REVIEWED."
- note added: "Z_{CABLE} ~40Ω Z_{PIC} termination has been simulated using IBIS models. Each output will need damping with discrete components at the LED strip."
- note removed: "If cable length requires it then place a further 4.7kΩ (externally) in parallel with R? and R? to increase the I^{2}C drive strength to about its maximum"
- note removed: "R?-?"
- note removed: "Z_{CABLE} ~40Ω Z_{PIC} termination simulated using IBIS."

Commit message: Finalised the schematic - checked over and added part numbers.  Ready for layout.
Parts:
- added D3: SD103AWS, restall-generic-sot:SOD-323, symbol restall-generic-diodes:schottky
- C12: Manufacturer (none) -> Wurth Elektronik; Manufacturer2 (none) -> Kyocera; Manufacturer2PartNumber (none) -> KGM05AR71E103KH; ManufacturerPartNumber (none) -> 885012205067
- C13: value 100nF -> 2.2μF; footprint restall-generic-capacitors:unpolarised-nominal-0402-1005 -> restall-generic-capacitors:unpolarised-nominal-0603-1608; Label 100nF±10% 10V X7R -> 2.2μF±10% 25V X7R; Manufacturer (none) -> Murata; Manufacturer2 (none) -> Murata; Manufacturer2PartNumber (none) -> GRM188Z71E225ME43D; ManufacturerPartNumber (none) -> GRM188Z71E225KE43D; Package 0402 -> 0603; VoltageRating 10V -> 25V
- C7: Manufacturer (none) -> Murata; Manufacturer2 (none) -> Cal-Chip Electronics; Manufacturer2PartNumber (none) -> GMC04X7R104K50NT; ManufacturerPartNumber (none) -> GRM155R71H104KE14J
- CONN1: footprint restall-generic-connectors:th-header-1x2-2.54mm-vertical -> (none)
- R1: renamed from R3; Manufacturer (none) -> Cal-Chip Electronics; Manufacturer2 (none) -> Yageo; Manufacturer2PartNumber (none) -> RC0402FR-1310KL; ManufacturerPartNumber (none) -> RM04F1002CT
- R10, R12, R31, R9: Manufacturer2 (none) -> Bourns; Manufacturer2PartNumber (none) -> CR0402-FX-6340GLF
- R11, R13, R32, R8: Manufacturer (none) -> Cal-Chip Electronics; Manufacturer2 (none) -> Yageo; Manufacturer2PartNumber (none) -> RC0402FR-1310KL; ManufacturerPartNumber (none) -> RM04F1002CT
- R14, R15, R16, R17, R18, R19, R20, R21: Manufacturer (none) -> Yageo; Manufacturer2 (none) -> Stackpole Electronics; Manufacturer2PartNumber (none) -> RMCF0402FT91R0; ManufacturerPartNumber (none) -> RC0402FR-0791RL
- R2: renamed from R4; value 1kΩ -> 910Ω; footprint restall-generic-resistors:nominal-0805-2012 -> restall-generic-resistors:nominal-1210-3225; Manufacturer (none) -> Stackpole Electronics; Manufacturer2 (none) -> Yageo; Manufacturer2PartNumber (none) -> RC1210FR-07910RL; ManufacturerPartNumber (none) -> RMCF1210FT910R; Package 0805 -> 1210; PowerRating 0.25W -> 0.4W
- R22, R23: Manufacturer (none) -> Walsin; Manufacturer2 (none) -> Yageo; Manufacturer2PartNumber (none) -> RC0402FR-134K7L; ManufacturerPartNumber (none) -> WR04X4701FTL
- R24: value 470Ω -> 634Ω; Label 470Ω±1% 0.0625W -> 634Ω±1% 0.0625W; Manufacturer (none) -> Yageo; Manufacturer2 (none) -> Bourns; Manufacturer2PartNumber (none) -> CR0402-FX-6340GLF; ManufacturerPartNumber (none) -> RC0402FR-07634RL
- R25: renamed from R27; Manufacturer2 (none) -> Bourns; Manufacturer2PartNumber (none) -> CR0402-FX-6340GLF
- R26: renamed from R28; Manufacturer2 (none) -> Bourns; Manufacturer2PartNumber (none) -> CR0402-FX-6340GLF
- R27: renamed from R29; Manufacturer2 (none) -> Bourns; Manufacturer2PartNumber (none) -> CR0402-FX-6340GLF
- R28: renamed from R30; Manufacturer2 (none) -> Bourns; Manufacturer2PartNumber (none) -> CR0402-FX-6340GLF
- R29: renamed from R25; Manufacturer (none) -> Walsin; Manufacturer2 (none) -> Yageo; Manufacturer2PartNumber (none) -> RC0402FR-134K7L; ManufacturerPartNumber (none) -> WR04X4701FTL
- R3: renamed from R1; Manufacturer (none) -> Bourns; Manufacturer2 (none) -> Yageo; Manufacturer2PartNumber (none) -> RC0402FR-0730K1L; ManufacturerPartNumber (none) -> CR0402-FX-3012GLF
- R30: renamed from R26; Manufacturer (none) -> Walsin; Manufacturer2 (none) -> Yageo; Manufacturer2PartNumber (none) -> RC0402FR-134K7L; ManufacturerPartNumber (none) -> WR04X4701FTL
- R4: renamed from R2; Manufacturer (none) -> Cal-Chip Electronics; Manufacturer2 (none) -> Yageo; Manufacturer2PartNumber (none) -> RC0402FR-1310KL; ManufacturerPartNumber (none) -> RM04F1002CT
- R5: Manufacturer (none) -> Walsin; Manufacturer2 (none) -> Bourns; Manufacturer2PartNumber (none) -> CR0402-FX-1003GLF; ManufacturerPartNumber (none) -> WR04X1003FTL
- R6: Manufacturer (none) -> Bourns; Manufacturer2 (none) -> Yageo; Manufacturer2PartNumber (none) -> RC0402FR-0730K1L; ManufacturerPartNumber (none) -> CR0402-FX-3012GLF
- R7: Manufacturer (none) -> Bourns; Manufacturer2 (none) -> Yageo; Manufacturer2PartNumber (none) -> RC0402FR-0752K3L; ManufacturerPartNumber (none) -> CR0402-FX-5232GLF
- renumbered D3 to D4, D4 to D5, D5 to D6
Connections:
- net +12V_{dc}: now also R3.1
- net +5Vdc: now also D3.1 (K)
- net VIN_{MON}: now also D3.2 (A)
- net at C1.1, CONN1.1 (P1), CONN1a.1 (P1)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: no longer R3.1
Other:
- note added: "PCB Stackup: L1 - Signal / Power L2 - Ground L3 - Ground L4 - Signal / Power JLC Stackup JLC04081H-7628: Z_{0}=40Ω, w=20.46mil, L1-L2 Z_{0}=85.25Ω, w=3.50mil, L1-L2"
- note added: "R25-28"
- note added: "Z_{0}=40Ω (20.46mil)"
- note removed: "R27-30"
- note removed: "TODO: NEEDS PROTECTION DIODE FROM C13 -> VCC, SINCE +12V COULD BE POWERED WHILST SMPS IS OFF !"
- note removed: "TODO: PART SELECTION STILL NEEDS TO BE DONE."
- note removed: "TODO: PIC BLOCK AND BLOCK TO RIGHT STILL TO REVIEW SMPS AND INPUT BLOCKS HAVE BEEN REVIEWED."
- moved on the sheet: C1, FB1, R3, R4, R5, R6
